File: hardware/remote-v2/sh1/knuth-gateway.sch (KiCad schematic (older format))
At the start: 22 parts, among them J1 FeatherLora1, J2 FeatherLora2, J3 Conn_01x02_Male, J6 Screw_Terminal_01x03, SW1 SW_SPDT, SW2 SW_SPDT

Commit message: update
Parts:
- added SW3: SW_SPDT, Connector_PinSocket_2.54mm:PinSocket_1x03_P2.54mm_Vertical, symbol Switch:SW_SPDT
Connections:
- net GND: now also SW3.2 (B); no longer D1.1 (K), D2.1 (K), D3.1 (K), D4.1 (K), D5.1 (K), D6.1 (K)
- new net: D1.1 (K), D2.1 (K), D3.1 (K), D4.1 (K), D5.1 (K), D6.1 (K), SW3.3 (C)
Changed lines of the file:
@@
 DI01
-$Comp
-L knuth-gateway-rescue:GND-power #PWR0102
-U 1 1 5E5EAD48
-P 3350 5050
-F 0 "#PWR0102" H 3350 4800 50  0001 C CNN
-F 1 "GND" H 3355 4877 50  0000 C CNN
-F 2 "" H 3350 5050 50  0001 C CNN
-F 3 "" H 3350 5050 50  0001 C CNN
-	1    3350 5050
-	1    0    0    -1
-$EndComp
 $Comp
 L knuth-gateway-rescue:R-Device R1
@@
 	1    0    0    -1
 $EndComp
-$Comp
-L knuth-gateway-rescue:GND-power #PWR0104
-U 1 1 5E5EFBCC
-P 3850 5050
-F 0 "#PWR0104" H 3850 4800 50  0001 C CNN
-F 1 "GND" H 3855 4877 50  0000 C CNN
-F 2 "" H 3850 5050 50  0001 C CNN
-F 3 "" H 3850 5050 50  0001 C CNN
-	1    3850 5050
-	1    0    0    -1
-$EndComp
-$Comp
-L knuth-gateway-rescue:GND-power #PWR0106
-U 1 1 5E5EFF0F
-P 4400 5050
-F 0 "#PWR0106" H 4400 4800 50  0001 C CNN
-F 1 "GND" H 4405 4877 50  0000 C CNN
-F 2 "" H 4400 5050 50  0001 C CNN
-F 3 "" H 4400 5050 50  0001 C CNN
-	1    4400 5050
-	1    0    0    -1
-$EndComp
-$Comp
-L knuth-gateway-rescue:GND-power #PWR0107
-U 1 1 5E5F021D
-P 4900 5050
-F 0 "#PWR0107" H 4900 4800 50  0001 C CNN
-F 1 "GND" H 4905 4877 50  0000 C CNN
-F 2 "" H 4900 5050 50  0001 C CNN
-F 3 "" H 4900 5050 50  0001 C CNN
-	1    4900 5050
-	1    0    0    -1
-$EndComp
-$Comp
-L knuth-gateway-rescue:GND-power #PWR0108
-U 1 1 5E5F1D45
-P 5400 5050
-F 0 "#PWR0108" H 5400 4800 50  0001 C CNN
-F 1 "GND" H 5405 4877 50  0000 C CNN
-F 2 "" H 5400 5050 50  0001 C CNN
-F 3 "" H 5400 5050 50  0001 C CNN
-	1    5400 5050
-	1    0    0    -1
-$EndComp
 Wire Wire Line
 	6200 3900 6800 3900
@@
 L knuth-gateway-rescue:GND-power #PWR0110
 U 1 1 5E6678FF
-P 2750 5050
-F 0 "#PWR0110" H 2750 4800 50  0001 C CNN
-F 1 "GND" H 2755 4877 50  0000 C CNN
-F 2 "" H 2750 5050 50  0001 C CNN
-F 3 "" H 2750 5050 50  0001 C CNN
-	1    2750 5050
+P 2000 4950
+F 0 "#PWR0110" H 2000 4700 50  0001 C CNN
+F 1 "GND" H 2005 4777 50  0000 C CNN
+F 2 "" H 2000 4950 50  0001 C CNN
+F 3 "" H 2000 4950 50  0001 C CNN
+	1    2000 4950
 	1    0    0    -1
 $EndComp
@@
 	1    0    0    -1
 $EndComp
+$Comp
+L Switch:SW_SPDT SW3
+U 1 1 5E61DD21
+P 2200 4950
+F 0 "SW3" H 2200 5235 50  0000 C CNN
+F 1 "SW_SPDT" H 2200 5144 50  0000 C CNN
+F 2 "Connector_PinSocket_2.54mm:PinSocket_1x03_P2.54mm_Vertical" H 2200 4950 50  0001 C CNN
+F 3 "~" H 2200 4950 50  0001 C CNN
+	1    2200 4950
+	1    0    0    -1
+$EndComp
+Wire Wire Line
+	5400 5050 4900 5050
+Wire Wire Line
+	4400 5050 4900 5050
+Connection ~ 4900 5050
+Wire Wire Line
+	4400 5050 3850 5050
+Connection ~ 4400 5050
+Wire Wire Line
+	3850 5050 3350 5050
+Connection ~ 3850 5050
+Wire Wire Line
+	3350 5050 2750 5050
+Connection ~ 3350 5050
+Wire Wire Line
+	2750 5050 2400 5050
+Connection ~ 2750 5050
 $EndSCHEMATC

Commit message: update
Parts:
- added H1, H2: MountingHole, MountingHole:MountingHole_2.7mm_M2.5, symbol Mechanical:MountingHole
- renumbered R2 to R1, R1 to R2
Changed lines of the file:
@@
 DI01
 $Comp
-L knuth-gateway-rescue:R-Device R1
+L knuth-gateway-rescue:R-Device R2
 U 1 1 5E5EA6D5
 P 3350 4600
-F 0 "R1" H 3420 4646 50  0000 L CNN
+F 0 "R2" H 3420 4646 50  0000 L CNN
 F 1 "1K" H 3420 4555 50  0000 L CNN
 F 2 "Resistor_THT:R_Axial_DIN0207_L6.3mm_D2.5mm_P2.54mm_Vertical" V 3280 4600 50  0001 C CNN
@@
 $EndComp
 $Comp
-L knuth-gateway-rescue:R-Device R2
+L knuth-gateway-rescue:R-Device R1
 U 1 1 5E667905
 P 2750 4600
-F 0 "R2" H 2820 4646 50  0000 L CNN
+F 0 "R1" H 2820 4646 50  0000 L CNN
 F 1 "1K" H 2820 4555 50  0000 L CNN
 F 2 "Resistor_THT:R_Axial_DIN0207_L6.3mm_D2.5mm_P2.54mm_Vertical" V 2680 4600 50  0001 C CNN
@@
 	2750 5050 2400 5050
 Connection ~ 2750 5050
+$Comp
+L Mechanical:MountingHole H1
+U 1 1 5E641806
+P 2950 950
+F 0 "H1" H 3050 996 50  0000 L CNN
+F 1 "MountingHole" H 3050 905 50  0000 L CNN
+F 2 "MountingHole:MountingHole_2.7mm_M2.5" H 2950 950 50  0001 C CNN
+F 3 "~" H 2950 950 50  0001 C CNN
+	1    2950 950
+	1    0    0    -1
+$EndComp
+$Comp
+L Mechanical:MountingHole H2
+U 1 1 5E641C08
+P 2950 1300
+F 0 "H2" H 3050 1346 50  0000 L CNN
+F 1 "MountingHole" H 3050 1255 50  0000 L CNN
+F 2 "MountingHole:MountingHole_2.7mm_M2.5" H 2950 1300 50  0001 C CNN
+F 3 "~" H 2950 1300 50  0001 C CNN
+	1    2950 1300
+	1    0    0    -1
+$EndComp
 $EndSCHEMATC

Commit message: final touches
Parts:
- renumbered RE3 to RSW
Connections:
- net +3V3: now also RSW.1; no longer SW2.1 (A)
- net GND: now also SW2.3 (C); no longer RSW.2
- new net: RSW.2, SW2.1 (A)
Other:
- moved on the sheet: RSW
Changed lines of the file:
@@
 A1
 $Comp
-L knuth-gateway-rescue:R-Device RE3
+L knuth-gateway-rescue:R-Device RSW
 U 1 1 5E5FA61D
-P 8250 1900
-F 0 "RE3" H 8320 1946 50  0000 L CNN
-F 1 "100K" H 8320 1855 50  0000 L CNN
-F 2 "Resistor_THT:R_Axial_DIN0207_L6.3mm_D2.5mm_P2.54mm_Vertical" V 8180 1900 50  0001 C CNN
-F 3 "~" H 8250 1900 50  0001 C CNN
-	1    8250 1900
+P 8250 1400
+F 0 "RSW" H 8320 1446 50  0000 L CNN
+F 1 "100K" H 8320 1355 50  0000 L CNN
+F 2 "Resistor_THT:R_Axial_DIN0207_L6.3mm_D2.5mm_P2.54mm_Vertical" V 8180 1400 50  0001 C CNN
+F 3 "~" H 8250 1400 50  0001 C CNN
+	1    8250 1400
 	1    0    0    -1
 $EndComp
@@
 L knuth-gateway-rescue:GND-power #PWR0113
 U 1 1 5E5FB986
-P 8250 2050
-F 0 "#PWR0113" H 8250 1800 50  0001 C CNN
-F 1 "GND" H 8255 1877 50  0000 C CNN
-F 2 "" H 8250 2050 50  0001 C CNN
-F 3 "" H 8250 2050 50  0001 C CNN
-	1    8250 2050
+P 8250 1750
+F 0 "#PWR0113" H 8250 1500 50  0001 C CNN
+F 1 "GND" H 8255 1577 50  0000 C CNN
+F 2 "" H 8250 1750 50  0001 C CNN
+F 3 "" H 8250 1750 50  0001 C CNN
+	1    8250 1750
 	1    0    0    -1
 $EndComp
@@
 L knuth-gateway-rescue:+3V3-power #PWR0114
 U 1 1 5E5FDE6D
-P 8250 1550
-F 0 "#PWR0114" H 8250 1400 50  0001 C CNN
-F 1 "+3V3" H 8265 1723 50  0000 C CNN
-F 2 "" H 8250 1550 50  0001 C CNN
-F 3 "" H 8250 1550 50  0001 C CNN
-	1    8250 1550
+P 8250 1250
+F 0 "#PWR0114" H 8250 1100 50  0001 C CNN
+F 1 "+3V3" H 8265 1423 50  0000 C CNN
+F 2 "" H 8250 1250 50  0001 C CNN
+F 3 "" H 8250 1250 50  0001 C CNN
+	1    8250 1250
 	1    0    0    -1
 $EndComp

Commit message: update
Parts:
- renumbered RSW to RSW1
Connections:
- net A2: now also R5.1
- net D6: no longer R5.1
Other:
- note added: "ACQUIRE"
- note added: "AWAKE"
- note added: "DATA"
- note added: "JOIN"
- note added: "SENT"
Changed lines of the file:
@@
 EESchema Schematic File Version 4
-EELAYER 30 0
+LIBS:knuth-gateway-cache
+EELAYER 29 0
 EELAYER END
 $Descr A4 11693 8268
@@
 	5400 4000 5400 4450
 Wire Wire Line
-	6200 3900 4900 3900
-Wire Wire Line
-	4900 3900 4900 4450
-Connection ~ 6200 3900
-Wire Wire Line
 	6200 3800 4400 3800
 Wire Wire Line
@@
 A1
 $Comp
-L knuth-gateway-rescue:R-Device RSW
+L knuth-gateway-rescue:R-Device RSW1
 U 1 1 5E5FA61D
 P 8250 1400
-F 0 "RSW" H 8320 1446 50  0000 L CNN
+F 0 "RSW1" H 8320 1446 50  0000 L CNN
 F 1 "100K" H 8320 1355 50  0000 L CNN
 F 2 "Resistor_THT:R_Axial_DIN0207_L6.3mm_D2.5mm_P2.54mm_Vertical" V 8180 1400 50  0001 C CNN
@@
 	1    0    0    -1
 $EndComp
+Text Notes 5000 5400 2    50   ~ 0
+JOIN
+Text Notes 4000 5400 2    50   ~ 0
+DATA
+Text Notes 3500 5400 2    50   ~ 0
+ACQUIRE
+Text Notes 2900 5400 2    50   ~ 0
+AWAKE
+Text Notes 4500 5400 2    50   ~ 0
+SENT
+Wire Wire Line
+	4900 4450 4900 4350
+Wire Wire Line
+	6650 4350 6650 3700
+Wire Wire Line
+	6650 3700 7350 3700
+Wire Wire Line
+	4900 4350 6650 4350
 $EndSCHEMATC
